File: hardware/snh/snh.kicad_sch (KiCad schematic)
At the start: 54 parts, among them J1 Trigger, J2 In, J3 Attenuverter In, J4 Out, J5 Smooth Out, J6 Attenuverter Out, J7 Pwr, Q1 BC547, SW1 SW_SPDT, U1 40106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

Commit message: Updating to mkdocs+material, generated BOM and schematic (small tweaks to clean up)
Parts:
- D3, D4: value D_Schottky -> 1N5819
Other:
- moved on the sheet: C16, C2, C3, C4, C5, C6, D1, D2, J2, J3, J4, J5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
